Commit message: {code integration}
Former-commit-id: adef72c2de7e200563622cd73fa40ffc9ce36bc0

File: install/slam/share/slam/urdf/slam2.urdf (robot description, URDF)
Before this commit: robot slam, 4 links, 3 joints
Links:
- removed link lidar_link
- added link base_footprint
- added link base_scan, mass 0.166931667241147; collision mesh filename=package://slam/meshes/lidar_link.STL; visual mesh filename=package://slam/meshes/lidar_link.STL
Joints:
- removed joint lidar_joint
- added joint base_joint: type fixed, parent base_footprint, child base_link, origin xyz=0 0 0.05 rpy=0 0 0
- added joint scan_joint: type fixed, parent base_link, child base_scan, origin xyz=0 0 0.856 rpy=0 0 0, axis 0 0 0
